File: hardware/slcam.kicad_sch (KiCad schematic)
At the start: 36 parts, among them J1 532610671, J2 Conn_01x08, J3 Conn_01x04, J4 532610371, J5 532610371, U1 STM32F103C8Tx, U2 W25Q128JVS, U3 TCAN330G, U4 TPS2044D, Y1 Crystal_GND24

Commit message: General fixes and improvements #45
Parts:
- removed XTAL?: ECS-.327-12.5-34R-C-TR, XTAL_ECX-34R_ECS, symbol ECS-327-12-5-34R-C-TR:ECS-.327-12.5-34R-C-TR
- added Y2: Crystal, lib:ECS-.327-12.5-34R-C-TR, symbol Device:Crystal
- C10, C9: footprint Capacitor_SMD:C_0603_1608Metric_Pad1.05x0.95mm_HandSolder -> Capacitor_SMD:C_0603_1608Metric_Pad1.08x0.95mm_HandSolder
Connections:
- net OSC_IN2: now also Y2.1
- net OSC_OUT2: now also Y2.2
Changed lines of the file:
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@@
     (stroke (width 0) (type default) (color 0 0 0 0))
   )
-  (wire (pts (xy 104.902 125.73) (xy 107.696 125.73))
+  (wire (pts (xy 104.902 125.73) (xy 108.966 125.73))
     (stroke (width 0) (type default) (color 0 0 0 0))
   )
@@
     (stroke (width 0) (type default) (color 0 0 0 0))
   )
-  (wire (pts (xy 117.856 125.73) (xy 120.65 125.73))
+  (wire (pts (xy 116.586 125.73) (xy 120.65 125.73))
     (stroke (width 0) (type default) (color 0 0 0 0))
   )
@@
       (effects (font (size 1.27 1.27)) (justify left))
     )
-    (property "Footprint" "Capacitor_SMD:C_0603_1608Metric_Pad1.05x0.95mm_HandSolder" (id 2) (at 121.6152 135.382 0)
+    (property "Footprint" "Capacitor_SMD:C_0603_1608Metric_Pad1.08x0.95mm_HandSolder" (id 2) (at 121.6152 135.382 0)
       (effects (font (size 1.27 1.27)) hide)
     )
     (property "Datasheet" "~" (id 3) (at 120.65 131.572 0)
       (effects (font (size 1.27 1.27)) hide)
-    )
-    (pin "1")
-    (pin "2")
-  )
-  (symbol (lib_id "ECS-327-12-5-34R-C-TR:ECS-.327-12.5-34R-C-TR") (at 117.856 125.73 180) (unit 1)
-    (in_bom yes) (on_board yes) (fields_autoplaced)
-    (property "Reference" "XTAL?" (id 0) (at 112.776 117.094 0)
-      (effects (font (size 1.524 1.524)))
-    )
-    (property "Value" "ECS-.327-12.5-34R-C-TR" (id 1) (at 112.776 120.904 0)
-      (effects (font (size 1.524 1.524)))
-    )
-    (property "Footprint" "XTAL_ECX-34R_ECS" (id 2) (at 112.776 116.586 0)
-      (effects (font (size 1.524 1.524)) hide)
-    )
-    (property "Datasheet" "" (id 3) (at 117.856 125.73 0)
-      (effects (font (size 1.524 1.524)))
     )
     (pin "1")
@@
       (effects (font (size 1.27 1.27)) (justify left))
     )
-    (property "Footprint" "Capacitor_SMD:C_0603_1608Metric_Pad1.05x0.95mm_HandSolder" (id 2) (at 105.8672 135.636 0)
+    (property "Footprint" "Capacitor_SMD:C_0603_1608Metric_Pad1.08x0.95mm_HandSolder" (id 2) (at 105.8672 135.636 0)
       (effects (font (size 1.27 1.27)) hide)
     )
     (property "Datasheet" "~" (id 3) (at 104.902 131.826 0)
+      (effects (font (size 1.27 1.27)) hide)
+    )
+    (pin "1")
+    (pin "2")
+  )
+  (symbol (lib_id "Device:Crystal") (at 112.776 125.73 0) (unit 1)
+    (in_bom yes) (on_board yes) (fields_autoplaced)
+    (property "Reference" "Y2" (id 0) (at 112.776 118.11 0))
+    (property "Value" "Crystal" (id 1) (at 112.776 120.65 0))
+    (property "Footprint" "lib:ECS-.327-12.5-34R-C-TR" (id 2) (at 112.776 125.73 0)
+      (effects (font (size 1.27 1.27)) hide)
+    )
+    (property "Datasheet" "~" (id 3) (at 112.776 125.73 0)
       (effects (font (size 1.27 1.27)) hide)
     )
@@
   (symbol (lib_name "GND_1") (lib_id "power:GND") (at 113.1097 135.636 0) (unit 1)
     (in_bom yes) (on_board yes) (fields_autoplaced)
-    (property "Reference" "#PWR?" (id 0) (at 113.1097 141.986 0)
+    (property "Reference" "#PWR0106" (id 0) (at 113.1097 141.986 0)
       (effects (font (size 1.27 1.27)) hide)
     )
@@
       (reference "#PWR0105") (unit 1) (value "VCC") (footprint "")
     )
+    (path "/d1fcd6c9-e9d6-4420-9597-c3534148d5df"
+      (reference "#PWR0106") (unit 1) (value "GND") (footprint "")
+    )
     (path "/8833683d-7a29-4916-8e0f-028e5284a8fd"
       (reference "#PWR0107") (unit 1) (value "GND") (footprint "")
@@
       (reference "#PWR0109") (unit 1) (value "GND") (footprint "")
     )
-    (path "/d1fcd6c9-e9d6-4420-9597-c3534148d5df"
-      (reference "#PWR?") (unit 1) (value "GND") (footprint "")
-    )
     (path "/00000000-0000-0000-0000-00006313d384"
       (reference "C1") (unit 1) (value "1uF") (footprint "Capacitor_SMD:C_0603_1608Metric_Pad1.05x0.95mm_HandSolder")
@@
     )
     (path "/b1256d30-6fd8-4cda-ac4e-1b9b06f9f7b6"
-      (reference "C9") (unit 1) (value "12pF") (footprint "Capacitor_SMD:C_0603_1608Metric_Pad1.05x0.95mm_HandSolder")
+      (reference "C9") (unit 1) (value "12pF") (footprint "Capacitor_SMD:C_0603_1608Metric_Pad1.08x0.95mm_HandSolder")
     )
     (path "/1c653fcf-bd3e-4143-82ac-50f37544835d"
-      (reference "C10") (unit 1) (value "12pF") (footprint "Capacitor_SMD:C_0603_1608Metric_Pad1.05x0.95mm_HandSolder")
+      (reference "C10") (unit 1) (value "12pF") (footprint "Capacitor_SMD:C_0603_1608Metric_Pad1.08x0.95mm_HandSolder")
     )
     (path "/00000000-0000-0000-0000-000063144f89"
@@
       (reference "U4") (unit 2) (value "TPS2044D") (footprint "Package_SO:SOIC-16_3.9x9.9mm_P1.27mm")
     )
-    (path "/2943a394-6d2a-4724-9337-7a8c8d89b171"
-      (reference "XTAL?") (unit 1) (value "ECS-.327-12.5-34R-C-TR") (footprint "XTAL_ECX-34R_ECS")
-    )
     (path "/00000000-0000-0000-0000-000062c8d4fe"
       (reference "Y1") (unit 1) (value "Crystal_GND24") (footprint "Crystal:Crystal_SMD_Abracon_ABM8G-4Pin_3.2x2.5mm")
     )
-  )
+    (path "/c55ccd54-28af-4ab4-883e-eafa97dc9bf8"
+      (reference "Y2") (unit 1) (value "Crystal") (footprint "lib:ECS-.327-12.5-34R-C-TR")
+    )
+  )
